File: Esp01Carrier.kicad_pcb (KiCad board)
At the start: 2 copper layers, 18.4 x 27.3 mm, 13 parts, among them P1 CONN_02X04, P2 CONN_01X07, P3 CONN_01X02, U1 LM317_SOT223

Commit message: updated to version III
Parts:
- removed REF** (x2): Symbol_OSHW-Logo_SilkScreen, Esp01:Symbol_OSHW-Logo_SilkScreen
- P3: value CONN_01X02 -> CONN_01X03; footprint Esp01:TerminalBlock_Pheonix_MKDS1.5-2pol -> Terminal_Blocks:TerminalBlock_Pheonix_MKDS1.5-3pol
- moved R3 6.63 mm to (130.2, 116.8)
- moved P3 5.08 mm to (132.1, 111.1)
Connections:
- C2 pad 1: Net-(C2-Pad1) -> VSS
- P3 pad 1: +3V3 -> VSS
- P3 pad 2: GND -> +3V3
- U1 pad 3: Net-(C2-Pad1) -> VSS
Routing:
- net +3V3: track 78.3 -> 57.8 mm, vias 0 -> 1
- net VSS: track 0.00 -> 16.7 mm, vias 0 -> 1
- net Net-(P1-Pad5): track 39.1 -> 24.7 mm, vias 0 -> 1
- net Net-(C2-Pad1): track 6.74 -> 0.00 mm
- net ESPRX: track 13.2 -> 14.8 mm, vias 0 -> 1
- net DTR: track 20.0 -> 20.8 mm
Other:
- board text added: "VIN"
- board text added: "Version III"
