File: Esp01Carrier.sch (KiCad schematic (older format))
At the start: 10 parts, among them P1 CONN_02X04, P2 CONN_01X07, P3 CONN_01X02, U1 LM317_SOT223

Commit message: updated to version III
Parts:
- removed P3: CONN_01X02, Esp01:TerminalBlock_Pheonix_MKDS1.5-2pol, symbol CONN_01X02
- added P3: CONN_01X03, Terminal_Blocks:TerminalBlock_Pheonix_MKDS1.5-3pol, symbol CONN_01X03
Connections:
- net +3V3: now also P3.2 (P2)
- net GND: now also P3.3 (P3)
- net VSS: now reaches C2.1, U1.3 (IN)
- net VSS: now also P3.1 (P1)
Changed lines of the file:
@@
 Connection ~ 6800 2150
 Wire Wire Line
-	6350 1200 6300 1200
+	6250 1200 6350 1200
 Wire Wire Line
 	6300 1200 6300 1850
@@
 Connection ~ 7750 1200
 $Comp
-L CONN_01X02 P3
-U 1 1 570954CE
-P 8350 3100
-F 0 "P3" H 8350 3250 50  0000 C CNN
-F 1 "CONN_01X02" V 8450 3100 50  0000 C CNN
-F 2 "Esp01:TerminalBlock_Pheonix_MKDS1.5-2pol" H 8350 3100 50  0001 C CNN
-F 3 "" H 8350 3100 50  0000 C CNN
-	1    8350 3100
-	1    0    0    -1
-$EndComp
-$Comp
 L +3.3V #PWR09
 U 1 1 5709555F
@@
 Wire Wire Line
 	5150 3200 5400 3200
-Text GLabel 6350 1400 3    60   Input ~ 0
+Text GLabel 6400 1500 3    60   Input ~ 0
 HEAT
 $Comp
@@
 	3450 3400 3400 3400
 Connection ~ 3400 3400
+$Comp
+L CONN_01X03 P3
+U 1 1 5724F79C
+P 8350 3050
+F 0 "P3" H 8350 3250 50  0000 C CNN
+F 1 "CONN_01X03" V 8450 3050 50  0000 C CNN
+F 2 "Terminal_Blocks:TerminalBlock_Pheonix_MKDS1.5-3pol" H 8350 3050 50  0001 C CNN
+F 3 "" H 8350 3050 50  0000 C CNN
+	1    8350 3050
+	1    0    0    -1
+$EndComp
+$Comp
+L VSS #PWR012
+U 1 1 5724F89A
+P 8050 2950
+F 0 "#PWR012" H 8050 2800 50  0001 C CNN
+F 1 "VSS" H 8050 3100 50  0000 C CNN
+F 2 "" H 8050 2950 50  0000 C CNN
+F 3 "" H 8050 2950 50  0000 C CNN
+	1    8050 2950
+	1    0    0    -1
+$EndComp
+$Comp
+L VSS #PWR013
+U 1 1 5724F906
+P 6250 1200
+F 0 "#PWR013" H 6250 1050 50  0001 C CNN
+F 1 "VSS" H 6250 1350 50  0000 C CNN
+F 2 "" H 6250 1200 50  0000 C CNN
+F 3 "" H 6250 1200 50  0000 C CNN
+	1    6250 1200
+	1    0    0    -1
+$EndComp
+Wire Wire Line
+	8050 2950 8150 2950
+Wire Wire Line
+	6350 1400 6350 1500
+Wire Wire Line
+	6350 1500 6400 1500
+Connection ~ 6300 1200
 $EndSCHEMATC
